File: sound laser.kicad_sch (KiCad schematic)
At the start: 10 parts, among them J1 AudioJack2, U1 L293DNE, U2 NE555P, U3 L7805

Commit message: rough wiring
Connections:
- net GND: now also R1.2, U1.12 (GND), U1.13 (GND), U1.4 (GND), U1.5 (GND), U3.2 (GND)
- net VCC: now also U1.16 (VCC1), U1.8 (VCC2), U3.1 (IN)
- net at LS1.2: now also U1.3 (1Y)
- net at R1.1: now also C1.2, U2.5 (CV)
- net at U1.1 (EN1,2): now also U3.3 (OUT)
- net at U1.2 (1A): now also U2.3 (Q)
Other:
- moved on the sheet: C1, C2, R1, R2, R3, U1, U2
